File: KiCad/V1/1DGames.kicad_sch (KiCad schematic)
At the start: 13 parts, among them J1 TM1637 Four Digits Led Displa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, Q1 AO3401A, Q2 AO3401A, U1 ESP32-DEVKITC-32D

Commit message: Fixed sound/buttons.
Parts:
- renumbered J1 to #J1
Connections:
- net +5V: now also Q1.3 (D)
- net SPEAKER_DRAIN: no longer Q1.3 (D)
Other:
- moved on the sheet: C1, Q2
